Commit message: Add simulation (#5)
* Add initial sim

* Add working robot description node, spawning robot still broken

* Add graded buoyancy and hydrodynamic forces

* Add lidar and camera sim bridge

* Add propellers

* Add temporarily working thrusters

* Redefine to catamaran, adjust hydrodynamic values

* Add IMU and GPS to sim

* Fix bug

* Update readme

* Remove static arg, raise lidar

* Add secondary world

* Add correct IMU transform

File: stinger_description/models/stinger_base/stinger_base.xacro (robot description, xacro)
@@ -1,118 +1,123 @@
 <?xml version="1.0"?>
 <robot xmlns:xacro="http://www.ros.org/wiki/xacro" name="stinger_base">
+    <xacro:include filename="$(find stinger_description)/models/stinger_base/components/sensors.xacro"/>
+    <xacro:include filename="$(find stinger_description)/models/stinger_base/components/thrusters.xacro"/>
     <xacro:macro name="stinger_base">
     <link name="hull_link">
       <inertial>
-        <pose>-0.05 0 -0.15 0 0 0</pose>
-        <mass value="30"/>
+        <pose>0.0 0.0 -0.13 0 0 0</pose>
+        <mass value="5"/>
         <inertia ixx="2.42369" ixy="0" ixz="0" iyy="3.9235025" iyz="0" izz="5.6403125"/>
       </inertial>
-      <collision>
-          <origin xyz="0 0 0.05" rpy="0 0 0"/>
-          <geometry>
-                <box size="0.381 0.204 0.135" />
-          </geometry>
-      </collision>
       <visual name="hull_visual">
+        <origin rpy="0 0 3.1416"/>
         <geometry>
-          <mesh filename="package://stinger_description/models/stinger_base/meshes/stinger_hull.dae"/>
-        </geometry>
-      </visual>
-      <visual name="motor_stbd_visual">
-        <geometry>
-          <mesh filename="package://stinger_description/models/stinger_base/meshes/stinger_prop.dae"/>
-        </geometry>
-      </visual>
-      <visual name="motor_port_visual">
-        <geometry>
-          <mesh filename="package://stinger_description/models/stinger_base/meshes/stinger_prop.dae"/>
+          <mesh filename="file://$(find stinger_description)/models/stinger_base/meshes/stinger_hull.dae"/>
         </geometry>
       </visual>
     </link>
-    <link name="camera_link">
-        <visual>
-            <origin xyz="-0.03 0 0" rpy="0 0 0"/>
-            <geometry>
-                <box size="0.06 0.15 0.15" />
-            </geometry>
-            <material name="white" />
-        </visual>
-        <visual>
-            <origin xyz="0.03 0 0" rpy="0 ${pi/2} 0"/>
-            <geometry>
-                <cylinder length="0.06" radius="0.04" />
-            </geometry>
-            <material name="blue" />
-        </visual>
-        <collision>
-            <origin xyz="0.0 0 0" rpy="0 0 0"/>
-            <geometry>
-                <box size="0.12 0.15 0.15" />
-            </geometry>
-        </collision>
-        <xacro:inertial_box mass="0.1" x="0.12" y="0.15" z="0.15">
-            <origin xyz="0.0 0 0" rpy="0 0 0"/>
-        </xacro:inertial_box>
+    <!-- port hull -->
+    <link name="hull_port_link">
+      <collision>
+          <origin xyz="0 0.0765 -0.05" rpy="0 0 0"/>
+          <geometry>
+                <box size="0.381 0.081 0.135" />
+          </geometry>
+      </collision>
     </link>
-    <joint name="camera_joint" type="fixed">
-        <origin xyz="0 0 0.1" rpy="0 0 0"/>
-        <parent link="hull_link"/>
-        <child link="camera_link"/>
-    </joint>
-    <link name="laser_frame">
-        <visual>
-            <geometry>
-                <cylinder radius="0.05" length="0.04"/>
-            </geometry>
-            <material name="red"/>
-        </visual>
-        <collision>
-            <geometry>
-                <cylinder radius="0.05" length="0.04"/>
-            </geometry>
-        </collision>
-        <xacro:inertial_cylinder mass="0.1" length="0.04" radius="0.05">
-            <origin xyz="0 0 0" rpy="0 0 0"/>
-        </xacro:inertial_cylinder>
-    </link>
-    <joint name="lidar_joint" type="fixed">
-        <origin xyz="0 0 0.1" rpy="0 0 0"/>
-        <parent link="hull_link"/>
-        <child link="lidar_link"/>
-    </joint>
-    <link name="imu_link">
-      <inertial>
-        <pose>0 0 0 0 0 0</pose>
-        <mass value="0.1"/>
-        <inertia ixx="0.0001" ixy="0" ixz="0" iyy="0.0001" iyz="0" izz="0.0001" />
-      </inertial>
-      <sensor name="imu_sensor" type="imu">
-        <pose degrees="true">0 0 0 180 0 0</pose>
-        <always_on>1</always_on>
-        <update_rate>1000.0</update_rate>
-      </sensor>
-    </link>
-    <joint name="imu_joint" type="fixed">
+    <joint name="hull_port_joint" type="fixed">
       <origin xyz="0 0 0"/>
       <parent link="hull_link"/>
-      <child link="imu_link"/>
+      <child link="hull_port_link"/>
     </joint>
-    <link name="gps_link">
-      <inertial>
-        <pose>0 0 0 0 0 0</pose>
-        <mass value="0.1"/>
-        <inertia ixx="0.0001" ixy="0" ixz="0" iyy="0.0001" iyz="0" izz="0.0001" />
-      </inertial>
-      <sensor name="gps_sensor" type="gps">
-        <pose degrees="true">0 0 0 180 0 0</pose>
-        <always_on>1</always_on>
-        <update_rate>1000.0</update_rate>
-      </sensor>
+    <!-- starboard hull -->
+    <link name="hull_stbd_link">
+      <collision>
+          <origin xyz="0 -0.0765 -0.05" rpy="0 0 0"/>
+          <geometry>
+                <box size="0.381 0.081 0.135" />
+          </geometry>
+      </collision>
     </link>
-    <joint name="gps_joint" type="fixed">
+    <joint name="hull_stbd_joint" type="fixed">
       <origin xyz="0 0 0"/>
       <parent link="hull_link"/>
-      <child link="gps_link"/>
+      <child link="hull_stbd_link"/>
     </joint>
+    <!-- Thrusters -->
+    <xacro:prop_macro thruster_id="port">
+      <origin xyz="-0.19 0.073 -0.041" rpy="0 0 0" />
+    </xacro:prop_macro>
+    <xacro:prop_macro thruster_id="stbd">
+      <origin xyz="-0.19 -0.073 -0.041 " rpy="0 0 0" />
+    </xacro:prop_macro>
+    <!-- Offset weight from propellers to maintain buoyancy -->
+    <!-- TODO: Find a better way to do this -->
+    <link name="box_offset_1">
+      <inertial>
+        <mass value="0.1" />
+        <origin xyz="0.19 0.073 -0.041" />
+        <inertia ixx="0.1" ixy="0.0" ixz="0.0"
+                iyy="0.1" iyz="0.0"
+                izz="0.1" />
+      </inertial>
+    </link>
+    <joint name="offset_joint_1" type="fixed">
+      <origin xyz="0 0 0"/>
+      <parent link="hull_link"/>
+      <child link="box_offset_1"/>
+    </joint>
+    <link name="box_offset_2">
+      <inertial>
+        <mass value="0.1" />
+        <origin xyz="0.19 -0.073 -0.041" />
+        <inertia ixx="0.1" ixy="0.0" ixz="0.0"
+                iyy="0.1" iyz="0.0"
+                izz="0.1" />
+      </inertial>
+    </link>
+    <joint name="offset_joint_2" type="fixed">
+      <origin xyz="0 0 0"/>
+      <parent link="hull_link"/>
+      <child link="box_offset_2"/>
+    </joint>
+    <!-- Sensors -->
+    <xacro:camera_macro camera_id="0">
+      <origin xyz="0.1 0 0" rpy="0 0 0" />
+    </xacro:camera_macro>
+    <xacro:lidar_macro>
+      <origin xyz="0.1 0 0.1" rpy="0 0 0" />
+    </xacro:lidar_macro>
+    <xacro:imu_macro>
+      <origin xyz="-0.05 0 0.025" rpy="3.14 0 0" />
+    </xacro:imu_macro>
+    <xacro:gps_macro>
+      <origin xyz="-0.05 0 0.025" rpy="0 0 0" />
+    </xacro:gps_macro>
+    <!-- hydrodynamics and control plugins -->
+    <gazebo>
+      <plugin
+        filename="gz-sim-hydrodynamics-system"
+        name="gz::sim::systems::Hydrodynamics">
+        <link_name> base_link </link_name>
+        <zW>-5.0</zW>
+        <zWabsW>-10.0</zWabsW>
+        <mQ>-50.0</mQ>
+        <mQabsQ>-100.0</mQabsQ>
+        <!-- Linear Drag -->
+        <xU>-5</xU> <!-- Surge -->
+        <yV>-5</yV> <!-- Sway -->
+        <zW>-5</zW> <!-- Heave -->
+        <kP>-10</kP> <!-- Roll-->
+        <mQ>-5</mQ> <!-- Pitch -->
+        <nR>-5</nR> <!-- Yaw-->
+        <xUabsU>-10</xUabsU>
+        <yVabsV>-60</yVabsV>
+        <zWabsW>-60</zWabsW>
+        <kPabsP>-10</kPabsP>
+        <mQabsQ>-60</mQabsQ>
+        <nRabsR>-50</nRabsR>
+      </plugin>
+    </gazebo>
     </xacro:macro>
 </robot>

Commit message: Fix camera transform and add grid world

File: stinger_description/models/stinger_base/stinger_base.xacro (robot description, xacro)
@@ -84,5 +84,5 @@
     <!-- Sensors -->
     <xacro:camera_macro camera_id="0">
-      <origin xyz="0.1 0 0" rpy="0 0 0" />
+      <origin xyz="0.16 0 0.012" rpy="0 0 0" />
     </xacro:camera_macro>
     <xacro:lidar_macro>
