Commit message: Fix hydrodynamics (#6)
* Fix hydrodynamics

* Fix typo

* Move mass into the hulls to add roll stability

File: stinger_description/models/stinger_base/components/thrusters.xacro (robot description, xacro)
@@ -13,7 +13,7 @@
       <!-- The inertial values need to be reasonable or gazebo will crash -->
       <inertial>
-        <mass value="0.1" />
-        <inertia ixx="0.01" ixy="0.0" ixz="0.0"
-                 iyy="0.01" iyz="0.0" izz="0.01" />
+        <mass value="0.0000001" />
+        <inertia ixx="0.00001" ixy="0.0" ixz="0.0"
+                 iyy="0.00001" iyz="0.0" izz="0.000001" />
       </inertial>
       <visual>

File: stinger_description/models/stinger_base/stinger_base.xacro (robot description, xacro)
@@ -7,6 +7,6 @@
       <inertial>
         <pose>0.0 0.0 -0.13 0 0 0</pose>
-        <mass value="5"/>
-        <inertia ixx="2.42369" ixy="0" ixz="0" iyy="3.9235025" iyz="0" izz="5.6403125"/>
+        <mass value="3"/>
+        <inertia ixx="1.42369" ixy="0" ixz="0" iyy="2.9235025" iyz="0" izz="3.6403125"/>
       </inertial>
       <visual name="hull_visual">
@@ -19,13 +19,24 @@
     <!-- port hull -->
     <link name="hull_port_link">
+      <inertial>
+        <mass value="1.0"/>
+        <inertia ixx="0.01" iyy="0.01" izz="0.01"
+                ixy="0.0" ixz="0.0" iyz="0.0"/>
+      </inertial>
       <collision>
-          <origin xyz="0 0.0765 -0.05" rpy="0 0 0"/>
-          <geometry>
-                <box size="0.381 0.081 0.135" />
-          </geometry>
+        <origin xyz="0.095 0.0 0.0" rpy="0 0 0"/>
+        <geometry>
+          <box size="0.19 0.081 0.135" />
+        </geometry>
+      </collision>
+      <collision>
+        <origin xyz="-0.095 0.0 0.0" rpy="0 0 0"/>
+        <geometry>
+          <box size="0.19 0.081 0.135" />
+        </geometry>
       </collision>
     </link>
     <joint name="hull_port_joint" type="fixed">
-      <origin xyz="0 0 0"/>
+      <origin xyz="0.0 0.0765 -0.035"/>
       <parent link="hull_link"/>
       <child link="hull_port_link"/>
@@ -33,13 +44,24 @@
     <!-- starboard hull -->
     <link name="hull_stbd_link">
+      <inertial>
+        <mass value="1.0"/>
+        <inertia ixx="0.01" iyy="0.01" izz="0.01"
+                ixy="0.0" ixz="0.0" iyz="0.0"/>
+      </inertial>
       <collision>
-          <origin xyz="0 -0.0765 -0.05" rpy="0 0 0"/>
-          <geometry>
-                <box size="0.381 0.081 0.135" />
+        <origin xyz="0.095 0 0" rpy="0 0 0"/>
+        <geometry>
+          <box size="0.19 0.081 0.135" />
+        </geometry>
+      </collision>
+      <collision>
+        <origin xyz="-0.095 0 0" rpy="0 0 0"/>
+        <geometry>
+          <box size="0.19 0.081 0.135" />
           </geometry>
       </collision>
     </link>
     <joint name="hull_stbd_joint" type="fixed">
-      <origin xyz="0 0 0"/>
+      <origin xyz="0.0 -0.0765 -0.035"/>
       <parent link="hull_link"/>
       <child link="hull_stbd_link"/>
@@ -50,36 +72,6 @@
     </xacro:prop_macro>
     <xacro:prop_macro thruster_id="stbd">
-      <origin xyz="-0.19 -0.073 -0.041 " rpy="0 0 0" />
+      <origin xyz="-0.19 -0.073 -0.041" rpy="0 0 0" />
     </xacro:prop_macro>
-    <!-- Offset weight from propellers to maintain buoyancy -->
-    <!-- TODO: Find a better way to do this -->
-    <link name="box_offset_1">
-      <inertial>
-        <mass value="0.1" />
-        <origin xyz="0.19 0.073 -0.041" />
-        <inertia ixx="0.1" ixy="0.0" ixz="0.0"
-                iyy="0.1" iyz="0.0"
-                izz="0.1" />
-      </inertial>
-    </link>
-    <joint name="offset_joint_1" type="fixed">
-      <origin xyz="0 0 0"/>
-      <parent link="hull_link"/>
-      <child link="box_offset_1"/>
-    </joint>
-    <link name="box_offset_2">
-      <inertial>
-        <mass value="0.1" />
-        <origin xyz="0.19 -0.073 -0.041" />
-        <inertia ixx="0.1" ixy="0.0" ixz="0.0"
-                iyy="0.1" iyz="0.0"
-                izz="0.1" />
-      </inertial>
-    </link>
-    <joint name="offset_joint_2" type="fixed">
-      <origin xyz="0 0 0"/>
-      <parent link="hull_link"/>
-      <child link="box_offset_2"/>
-    </joint>
     <!-- Sensors -->
     <xacro:camera_macro camera_id="0">
@@ -101,8 +93,4 @@
         name="gz::sim::systems::Hydrodynamics">
         <link_name> base_link </link_name>
-        <zW>-5.0</zW>
-        <zWabsW>-10.0</zWabsW>
-        <mQ>-50.0</mQ>
-        <mQabsQ>-100.0</mQabsQ>
         <!-- Linear Drag -->
         <xU>-5</xU> <!-- Surge -->
@@ -119,4 +107,10 @@
         <nRabsR>-50</nRabsR>
       </plugin>
+      <!-- Publishes perfect odometry data for ground truth -->
+      <plugin
+        filename="gz-sim-odometry-publisher-system"
+        name="gz::sim::systems::OdometryPublisher">
+        <dimensions>3</dimensions>
+      </plugin>
     </gazebo>
     </xacro:macro>
