Commit message: Sync from private repo (answers folder removed, .github ignored)

File: stinger_description/models/stinger_base/components/sensors.xacro (robot description, xacro)
@@ -63,5 +63,4 @@
         <visualize>true</visualize>
         <topic>stinger/laser/scan</topic>
-        <!-- This tag isn't recognized by SDF but is extremely important for getting the correct TF data for the sonar frame-->
         <gz_frame_id>lidar</gz_frame_id>
       </sensor>
@@ -69,12 +68,12 @@
   </xacro:macro>
   <xacro:macro name="imu_macro" params="*origin">
-    <link name="imu"/>
+    <link name="imu_link"/>
     <joint name="imu_joint" type="fixed">
       <xacro:insert_block name="origin"/>
-      <parent link="hull_link"/>
-      <child link="imu"/>
+      <parent link="base_link"/>
+      <child link="imu_link"/>
       <axis xyz="1 0 0"/>
     </joint>
-    <gazebo reference="imu">
+    <gazebo reference="imu_link">
       <sensor name="imu_sensor" type="imu">
         <pose>0 0 0 0 0 0</pose>
@@ -84,5 +83,5 @@
         <update_rate>1000</update_rate>
         <!-- This tag isn't recognized by SDF but is extremely important for getting the correct TF data for the IMU frame-->
-        <gz_frame_id>imu</gz_frame_id>
+        <gz_frame_id>imu_link</gz_frame_id>
       </sensor>
     </gazebo>
@@ -100,5 +99,5 @@
         <update_rate>10</update_rate>
         <topic>stinger/gps/fix</topic>
-        <gz_frame_id>gps</gz_frame_id>
+        <gz_frame_id>gps_link</gz_frame_id>
       </sensor>
     </gazebo>
